Commit message: Fixed translation issues for the z lift

File: ur10e_mod/urdf/ur10e_mod_gz.urdf.xacro (robot description, xacro)
@@ -20,37 +20,41 @@
   <!-- World -->
   <link name="world"/>
+  <link name="base_prismatic_link">
+    <inertial>
+      <mass value="10.0"/>
+      <inertia ixx="0.1" ixy="0.0" ixz="0.0" iyy="0.1" iyz="0.0" izz="0.1"/>
+    </inertial>
+  </link>
+  <joint name="base_prismatic_joint" type="fixed">
+    <parent link="world"/>
+    <child link="base_prismatic_link"/>
+  </joint>
   <!-- Prismatic Lift -->
   <link name="z_lift_link">
     <visual>
-        <geometry>
-        <cylinder radius="0.1" length="0.05"/>
-        </geometry>
-        <origin xyz="0 0 0.025" rpy="0 0 0"/>
+      <geometry>
+        <cylinder length="0.05" radius="0.1"/>
+      </geometry>
+      <origin rpy="0 0 0" xyz="0 0 0.025"/>
     </visual>
+    <collision>
+      <geometry>
+        <cylinder length="0.05" radius="0.1"/>
+      </geometry>
+      <origin rpy="0 0 0" xyz="0 0 0.025"/>
+    </collision>
     <inertial>
-        <mass value="1.0"/>
-        <origin xyz="0 0 0.025" rpy="0 0 0"/>
-        <inertia ixx="0.01" ixy="0.0" ixz="0.0"
-                iyy="0.01" iyz="0.0"
-                izz="0.01"/>
+      <mass value="1.0"/>
+      <origin rpy="0 0 0" xyz="0 0 0.025"/>
+      <inertia ixx="0.01" ixy="0.0" ixz="0.0" iyy="0.01" iyz="0.0" izz="0.01"/>
     </inertial>
   </link>
   <joint name="z_lift_joint" type="prismatic">
-    <parent link="world"/>
+    <parent link="base_prismatic_link"/>
     <child link="z_lift_link"/>
     <origin xyz="0 0 0" rpy="0 0 0"/>
     <axis xyz="0 0 1"/>
-    <limit lower="0.0" upper="1.0" effort="100" velocity="0.2"/>
+    <limit lower="0.0" upper="1.0" effort="1000" velocity="1.0"/>
   </joint>
-  <!-- Transmission -->
-  <transmission name="z_lift_trans">
-    <type>transmission_interface/SimpleTransmission</type>
-    <joint name="z_lift_joint">
-      <hardwareInterface>position</hardwareInterface>
-    </joint>
-    <actuator name="z_lift_motor">
-      <mechanicalReduction>1.0</mechanicalReduction>
-    </actuator>
-  </transmission>
   <!-- Arm -->
   <xacro:ur_robot
@@ -69,14 +73,9 @@
   </xacro:ur_robot>
   <!-- Gazebo Plugin -->
-  <gazebo>
-    <plugin filename="libgz_ros2_control-system.so" name="gz_ros2_control::GazeboSimROS2ControlPlugin">
-      <parameters>$(find ur10e_mod)/config/ur_controllers_with_z_lift.yaml</parameters>
-    </plugin>
-  </gazebo>
   <gazebo reference="world">
   </gazebo>
   <gazebo>
     <plugin filename="gz_ros2_control-system" name="gz_ros2_control::GazeboSimROS2ControlPlugin">
-      <parameters>$(arg simulation_controllers)</parameters>
+      <parameters>$(find ur10e_mod)/config/ur_controllers_with_z_lift.yaml</parameters>
       <ros>
         <namespace>$(arg ros_namespace)</namespace>

Commit message: Explicitly add config files for the ur10e robot

File: ur10e_mod/urdf/ur10e_mod_gz.urdf.xacro (robot description, xacro)
@@ -5,8 +5,8 @@
   <xacro:arg name="tf_prefix" default=""/>
   <xacro:arg name="ur_type" default="ur10e"/>
-  <xacro:arg name="joint_limit_params" default="$(find ur_description)/config/$(arg ur_type)/joint_limits.yaml"/>
-  <xacro:arg name="kinematics_params" default="$(find ur_description)/config/$(arg ur_type)/default_kinematics.yaml"/>
-  <xacro:arg name="physical_params" default="$(find ur_description)/config/$(arg ur_type)/physical_parameters.yaml"/>
-  <xacro:arg name="visual_params" default="$(find ur_description)/config/$(arg ur_type)/visual_parameters.yaml"/>
+  <xacro:arg name="joint_limit_params" default="$(find ur10e_mod)/config/joint_limits.yaml"/>
+  <xacro:arg name="kinematics_params" default="$(find ur10e_mod)/config/default_kinematics.yaml"/>
+  <xacro:arg name="physical_params" default="$(find ur10e_mod)/config/physical_parameters.yaml"/>
+  <xacro:arg name="visual_params" default="$(find ur10e_mod)/config/visual_parameters.yaml"/>
   <xacro:arg name="safety_limits" default="false"/>
   <xacro:arg name="safety_pos_margin" default="0.15"/>
@@ -55,5 +55,5 @@
     <origin xyz="0 0 0" rpy="0 0 0"/>
     <axis xyz="0 0 1"/>
-    <limit lower="0.0" upper="1.0" effort="1000" velocity="1.0"/>
+    <limit lower="0.0" upper="1.0" effort="10000" velocity="1.0"/>
   </joint>
   <!-- Arm -->

Commit message: Add visual elements for the prismatic joint

File: ur10e_mod/urdf/ur10e_mod_gz.urdf.xacro (robot description, xacro)
@@ -21,4 +21,13 @@
   <link name="world"/>
   <link name="base_prismatic_link">
+    <visual>
+      <origin xyz="0.0 -0.125 0.525" rpy="0 0 0"/>
+      <geometry>
+        <box size="0.25 0.05 1.05"/>
+      </geometry>
+      <material name="grey">
+        <color rgba="0.6 0.6 0.6 0.5"/>
+      </material>
+    </visual>
     <inertial>
       <mass value="10.0"/>
@@ -33,8 +42,11 @@
   <link name="z_lift_link">
     <visual>
+      <origin xyz="0.0 0.0 0.025" rpy="0 0 0"/>
       <geometry>
-        <cylinder length="0.05" radius="0.1"/>
+        <box size="0.2 0.2 0.05"/>
       </geometry>
-      <origin rpy="0 0 0" xyz="0 0 0.025"/>
+      <material name="red">
+        <color rgba="0 0 0 0.75"/>
+      </material>
     </visual>
     <collision>
